Commit message: gripper link to plan  and execute trajectory based on that link

File: robotiq_85_description/urdf/robotiq_85_gripper.urdf.xacro (robot description, xacro)
@@ -2,4 +2,10 @@
 <robot name="robotiq_85_gripper" xmlns:xacro="http://ros.org/wiki/xacro">
     <xacro:include filename="$(find robotiq_85_description)/urdf/robotiq_85_gripper.transmission.xacro" />
+    <!-- geometry macros for modeling geometric primitives with according meshes -->
+    <xacro:macro name="sphere_geometry" params="radius">
+      <geometry>
+        <mesh filename="package://robotiq_85_description/meshes/unit_sphere.stl" scale="${radius} ${radius} ${radius}"/>
+      </geometry>
+    </xacro:macro>
     <xacro:macro name="robotiq_85_gripper" params="prefix parent *origin">
         <joint name="${prefix}gripper_base_joint" type="fixed">
@@ -299,4 +305,27 @@
             <kd>1.0</kd>
         </gazebo>
+	<joint name="gripper_to_tcp" type="fixed">
+	    <parent link="${prefix}gripper_base_link"/>
+            <child link="${prefix}gripper"/>
+            <origin xyz=" 0.1500 0.0 0.0" rpy="3.1415 0 0"/>
+        </joint>
+	<link name="${prefix}gripper">
+            <visual>
+                <xacro:sphere_geometry radius="0.005"/>
+                <material name="white">
+                    <color rgba="1 1 1 0.5"/>
+                </material>
+            </visual>
+            <collision>
+                <xacro:sphere_geometry radius="0.005"/>
+            </collision>
+	</link>
+        <gazebo reference="${prefix}gripper">
+            <implicitSpringDamper>1</implicitSpringDamper>
+            <mu1>100000</mu1>
+            <mu2>100000</mu2>
+            <kp>100000000.0</kp>
+            <kd>1.0</kd>
+        </gazebo>
         <xacro:robotiq_85_gripper_transmission prefix="${prefix}" />
     </xacro:macro>
